Commit message: 2025/10/10_14:03 update navigation2

File: 1_URDF_ws/install/robot/share/robot/urdf/robot/actor/wheel_congdong.urdf.xacro (robot description, xacro)
@@ -40,5 +40,5 @@
         <!-- 机器人的关节：组合机器人部件 -->
         <!-- wheel是活动的，所以使用"continuous" -->
-        <joint name="${wheel_name}_joint" type="revolute">
+        <joint name="${wheel_name}_joint" type="continuous">
             <!-- 表示把wheel固定到机器人上 -->
             <parent link="base_link"/>
@@ -51,6 +51,6 @@
         </joint>
         <gazebo reference="${wheel_name}_link">
-            <mu1 value="0.0"/>   <!-- 切向摩擦系数 -->
-            <mu2 value="0.0"/>   <!-- 法向摩擦系数 -->
+            <mu1 value="5.0"/>   <!-- 切向摩擦系数 -->
+            <mu2 value="5.0"/>   <!-- 法向摩擦系数 -->
             <kp value="1000000000.0"/> <!-- 刚度擦系数 -->
             <kd value="1.0"/>     <!-- 阻尼系数 -->

File: 1_URDF_ws/install/robot/share/robot/urdf/robot/plugins/gazebo_control_plugin.xacro (robot description, xacro)
@@ -26,5 +26,5 @@
                 <!-- 决定是否发布某些话题 -->
                 <publish_odom>true</publish_odom>
-                <publish_odom_tf>ytue</publish_odom_tf>
+                <publish_odom_tf>true</publish_odom_tf>
                 <publish_wheel_tf>true</publish_wheel_tf>
                 <odometry_frame>odom</odometry_frame>
